Commit message: gazebo

File: mrobot_gazebo/urdf/loui_robot_body.urdf.xacro (robot description, xacro)
@@ -27,5 +27,5 @@
     <xacro:property name="motor_x" value="0.12"/>
     <!-- Caster radius and mass -->
-    <xacro:property name="caster_radius"          value="0.027" />
+    <xacro:property name="caster_radius"          value="0.025" />
     <xacro:property name="caster_mass"            value="0.017" />
     <xacro:property name="caster_joint_origin_x"  value="-0.21" />
@@ -125,5 +125,5 @@
             <parent link="base_link"/>
             <child link="${fb}_caster_link"/>
-            <origin xyz="${translateX*caster_joint_origin_x} 0 ${-caster_radius}" rpy="0 0 0"/>
+            <origin xyz="${translateX*caster_joint_origin_x} 0 ${-caster_radius-base_link_height/2}" rpy="0 0 0"/>
         </joint>
     </xacro:macro>
@@ -245,9 +245,9 @@
                 <publishWheelJointState>true</publishWheelJointState>
                 <alwaysOn>true</alwaysOn>
-                <updateRate>100.0</updateRate>
+                <updateRate>200.0</updateRate>
                 <legacyMode>true</legacyMode>
                 <leftJoint>base_to_wheel_left_joint</leftJoint>
                 <rightJoint>base_to_wheel_right_joint</rightJoint>
-                <wheelSeparation>${base_link_width}</wheelSeparation>
+                <wheelSeparation>${base_link_width+wheel_height}</wheelSeparation>
                 <wheelDiameter>${2*wheel_radius}</wheelDiameter>
                 <broadcastTF>1</broadcastTF>

File: mrobot_gazebo/urdf/loui_robot_with_camera_imu.urdf.xacro (robot description, xacro)
@@ -3,7 +3,12 @@
 	<xacro:include filename="$(find mrobot_gazebo)/urdf/loui_robot_body.urdf.xacro" />
 	<xacro:include filename="$(find mrobot_gazebo)/urdf/camera.xacro" />
+	<xacro:include filename="$(find mrobot_gazebo)/urdf/imu.xacro" />
 	<xacro:property name="camera_offset_x" value="0.21" />
 	<xacro:property name="camera_offset_y" value="0" />
 	<xacro:property name="camera_offset_z" value="0.02" />
+	<!-- imu parameter:0.12 0 0.005 -->
+	<xacro:property name="imu_offset_x" value="0.12" />
+	<xacro:property name="imu_offset_y" value="0.0" />
+	<xacro:property name="imu_offset_z" value="0.005" />
 	<!-- Body of mrobot, with plates, standoffs and Create (including sim sensors) -->
 	<mrobot_body/>
@@ -15,3 +20,9 @@
 	</joint>
 	<xacro:usb_camera prefix="camera"/>
+	<joint name="imu_joint" type="fixed">
+		<origin xyz="${imu_offset_x} ${imu_offset_y} ${imu_offset_z}" rpy="0 0 0" />
+		<parent link="base_link"/>
+		<child link="imu_link"/>
+	</joint>
+	<xacro:imu prefix="imu"/>
 </robot>
