Commit message: imu test

File: mrobot_gazebo/urdf/loui_robot_with_camera_imu.urdf.xacro (robot description, xacro)
@@ -10,5 +10,5 @@
 	<xacro:property name="imu_offset_x" value="0.12" />
 	<xacro:property name="imu_offset_y" value="0.0" />
-	<xacro:property name="imu_offset_z" value="0.005" />
+	<xacro:property name="imu_offset_z" value="0.05" />
 	<!-- Body of mrobot, with plates, standoffs and Create (including sim sensors) -->
 	<mrobot_body/>
